Commit message: update self collision model for autolife

File: assets/autolife/autolife_spherized.urdf (robot description, URDF)
Before this commit: robot autolife, 37 links, 36 joints
Links:
- link Joint_Left_Gripper_Left_Finger: geometry collision sphere radius=0.009927; collision sphere radius=0.012328
- link Link_Ankle_to_Knee: geometry collision sphere radius=0.104948; collision sphere radius=0.109059
- link Link_Chest_Back_Cover: geometry collision sphere radius=0.053563; collision sphere radius=0.054873
- link Link_Chest_Front_Cover: geometry collision sphere radius=0.039871; collision sphere radius=0.042146
- link Link_Ground_Vehicle_Visual_Cover: geometry collision sphere radius=0.088961; collision sphere radius=0.093048
- link Link_Ground_Vehicle_Z: geometry collision sphere radius=0.126008; collision sphere radius=0.130365
- link Link_Knee_Black_Cover: geometry collision sphere radius=0.074351; collision sphere radius=0.074489
- link Link_Knee_to_Waist_Pitch: geometry collision sphere radius=0.076283; collision sphere radius=0.079998
- link Link_Left_Elbow_to_Forearm: geometry collision sphere radius=0.028661; collision sphere radius=0.041523
- link Link_Left_Forearm_to_Wrist_Upper: geometry collision sphere radius=0.026535; collision sphere radius=0.027497
- link Link_Left_Gripper: geometry collision sphere radius=0.012335; collision sphere radius=0.013899
- link Link_Left_Gripper_Left_Inner_Knuckle: geometry collision sphere radius=0.00765; collision sphere radius=0.009212
- link Link_Left_Gripper_Right_Finger: geometry collision sphere radius=0.010833; collision sphere radius=0.012044
- link Link_Left_Gripper_Right_Inner_Knuckle: geometry collision sphere radius=0.00984; collision sphere radius=0.010462
- link Link_Left_Gripper_Right_Outer_Knuckle: geometry collision sphere radius=0.013998; collision sphere radius=0.014081
- link Link_Left_Shoulder_Inner_to_Shoulder_Outer: geometry collision sphere radius=0.05919; collision sphere radius=0.059314
- link Link_Left_Shoulder_Outer_to_UpperArm: geometry collision sphere radius=0.030168; collision sphere radius=0.044751
- link Link_Left_UpperArm_to_Elbow: geometry collision sphere radius=0.042576; collision sphere radius=0.049773
- link Link_Left_Wrist_Lower_to_Gripper: geometry collision sphere radius=0.022526; collision sphere radius=0.024141
- link Link_Left_Wrist_Upper_to_Wrist_Lower: geometry collision sphere radius=0.042266; collision sphere radius=0.042426
- link Link_Mask: geometry collision sphere radius=0.043435; collision sphere radius=0.045536
- link Link_Right_Elbow_to_Forearm: geometry collision sphere radius=0.023299; collision sphere radius=0.023362
- link Link_Right_Forearm_to_Wrist_Upper: geometry collision sphere radius=0.026535; collision sphere radius=0.027497
- link Link_Right_Gripper: geometry collision sphere radius=0.012335; collision sphere radius=0.013899
- link Link_Right_Gripper_Left_Finger: geometry collision sphere radius=0.009927; collision sphere radius=0.012328
- link Link_Right_Gripper_Left_Inner_Knuckle: geometry collision sphere radius=0.00765; collision sphere radius=0.009212
- link Link_Right_Gripper_Right_Finger: geometry collision sphere radius=0.010833; collision sphere radius=0.012044
- link Link_Right_Gripper_Right_Inner_Knuckle: geometry collision sphere radius=0.009674; collision sphere radius=0.011852
- link Link_Right_Gripper_Right_Outer_Knuckle: geometry collision sphere radius=0.013998; collision sphere radius=0.014081
- link Link_Right_Shoulder_Outer_to_UpperArm: geometry collision sphere radius=0.050119; collision sphere radius=0.051464
- link Link_Right_UpperArm_to_Elbow: geometry collision sphere radius=0.042576; collision sphere radius=0.049773
- link Link_Right_Wrist_Lower_to_Gripper: geometry collision sphere radius=0.023596; collision sphere radius=0.024495
- link Link_Right_Wrist_Upper_to_Wrist_Lower : geometry collision sphere radius=0.042266; collision sphere radius=0.042426
- link Link_Waist_Pitch_to_Waist_Yaw: geometry collision sphere radius=0.064651; collision sphere radius=0.066208
- link Link_Waist_Yaw_to_Shoulder_Inner: geometry collision sphere radius=0.079736; collision sphere radius=0.103716
